File: r1/src/tr25-sao-r1/tr25-sao-r1.kicad_pcb (KiCad board)
At the start: 0 parts

Commit message: Mask tractor beam
Parts:
- added N1: Housing, tr25-sao:tr25, F.Cu at (77.6, 98.6)
Other:
- board outline added: 46.8 x 68 mm
- copper layers 0 -> 2
